Commit message: Modified Joint Angles
Can now use proper joint angle visualization, changes joint positions to match assignment.

File: rrbot_description/urdf/rrbot.xacro (robot description, xacro)
@@ -113,6 +113,6 @@
     <child link="link4"/>
     <origin xyz="${width2} 0 ${height2}" rpy="0 0 0"/>
-    <axis xyz="0 0 1"/>
-    <limit effort="0.1" lower="-.5" upper="0" velocity="0.15"/>
+    <axis xyz="0 0 -1"/>
+    <limit effort="0.5" lower="-.01" upper=".99" velocity="0.15"/>
   </joint>
  <link name="link4">

Commit message: Add files via upload
Modified effort values

File: rrbot_description/urdf/rrbot.xacro (robot description, xacro)
@@ -47,5 +47,5 @@
     </inertial>
   </link>
-  <joint name="joint1" type="continuous">
+  <joint name="joint1" type="revolute">
     <parent link="link1"/>
     <child link="link2"/>
@@ -53,4 +53,5 @@
     <axis xyz="0 0 1"/>
     <dynamics damping="0.7"/>
+     <limit effort="80" lower="-3.141" upper="3.141" velocity="0.15"/>
   </joint>
   <!-- Middle Link -->
@@ -78,9 +79,10 @@
     </inertial>
   </link>
-  <joint name="joint2" type="continuous">
+  <joint name="joint2" type="revolute">
     <parent link="link2"/>
     <child link="link3"/>
     <origin xyz="${width2/2} 0 ${height2}" rpy="0 0 0"/>
     <axis xyz="0 0 1"/>
+    <limit effort="80" lower="-3.141" upper="3.141" velocity="0.15"/>
     <dynamics damping="0.7"/>
   </joint>
@@ -114,5 +116,5 @@
     <origin xyz="${width2} 0 ${height2}" rpy="0 0 0"/>
     <axis xyz="0 0 -1"/>
-    <limit effort="0.5" lower="-.01" upper=".99" velocity="0.15"/>
+    <limit effort="80" lower="-.01" upper=".99" velocity="0.15"/>
   </joint>
  <link name="link4">
@@ -159,3 +161,13 @@
     </actuator>
   </transmission>
+  <transmission name="tran3">
+    <type>transmission_interface/SimpleTransmission</type>
+    <joint name="joint3">
+      <hardwareInterface>hardware_interface/EffortJointInterface</hardwareInterface>
+    </joint>
+    <actuator name="motor3">
+      <hardwareInterface>hardware_interface/EffortJointInterface</hardwareInterface>
+      <mechanicalReduction>1</mechanicalReduction>
+    </actuator>
+  </transmission>
 </robot>
